File: Pre-amp/Pre-amp.sch (KiCad schematic (older format))
At the start: 52 parts, among them J1 In, J2 Send, J3 Return, J4 Out, J5 PWR, U1 LF353N, U2 LF353N, U3 LF353N

Commit message: Add buffer input to pre-amp
Parts:
- added C1: .1, Capacitor_THT:C_Disc_D3.8mm_W2.6mm_P2.50mm, symbol Device:C
- added C2: 100pf, Capacitor_THT:C_Disc_D3.8mm_W2.6mm_P2.50mm, symbol Device:C
- added C3: 10µF, Capacitor_THT:CP_Radial_D4.0mm_P1.50mm, symbol Device:CP
- added C4: .22, Capacitor_THT:C_Disc_D3.8mm_W2.6mm_P2.50mm, symbol Device:C
- added C5: .0033, Capacitor_THT:C_Disc_D3.8mm_W2.6mm_P2.50mm, symbol Device:C
- added C6: 10, Capacitor_THT:C_Disc_D3.8mm_W2.6mm_P2.50mm, symbol Device:C
- added D1, D2: 1N759, Diode_THT:D_DO-35_SOD27_P7.62mm_Horizontal, symbol Device:D_Zener
- added H3, H4: MountingHole, MountingHole:MountingHole_2.2mm_M2_DIN965_Pad, symbol Mechanical:MountingHole
- added R1, R5: 33k, Resistor_THT:R_Axial_DIN0207_L6.3mm_D2.5mm_P7.62mm_Horizontal, symbol Device:R
- added R10, R11, R7: 22k, Resistor_THT:R_Axial_DIN0207_L6.3mm_D2.5mm_P7.62mm_Horizontal, symbol Device:R
- added R12, R9: 1k, Resistor_THT:R_Axial_DIN0207_L6.3mm_D2.5mm_P7.62mm_Horizontal, symbol Device:R
- added R13: 82k, Resistor_THT:R_Axial_DIN0207_L6.3mm_D2.5mm_P7.62mm_Horizontal, symbol Device:R
- added R14, R4, R6: 3.3k, Resistor_THT:R_Axial_DIN0207_L6.3mm_D2.5mm_P7.62mm_Horizontal, symbol Device:R
- added R2: 23k, Resistor_THT:R_Axial_DIN0207_L6.3mm_D2.5mm_P7.62mm_Horizontal, symbol Device:R
- added R3: 220k, Resistor_THT:R_Axial_DIN0207_L6.3mm_D2.5mm_P7.62mm_Horizontal, symbol Device:R
- added R8: 12k, Resistor_THT:R_Axial_DIN0207_L6.3mm_D2.5mm_P7.62mm_Horizontal, symbol Device:R
- added RV1: 25k-L, Potentiometer_THT:Potentiometer_ACP_CA9-H2,5_Horizontal, symbol Device:R_POT_US
- added U1: LF353N, Package_DIP:DIP-8_W7.62mm_LongPads, symbol Pre-amp-rescue:LF353N-2019-03-05_16-55-55
- C10: renamed from C4; footprint Capacitors_THT:C_Axial_L3.8mm_D2.6mm_P7.50mm_Horizontal -> Capacitor_THT:C_Disc_D3.8mm_W2.6mm_P2.50mm
- C11: renamed from C5; footprint Capacitors_THT:C_Axial_L3.8mm_D2.6mm_P7.50mm_Horizontal -> Capacitor_THT:C_Disc_D3.8mm_W2.6mm_P2.50mm
- C12: renamed from C6; footprint Capacitors_THT:C_Axial_L3.8mm_D2.6mm_P7.50mm_Horizontal -> Capacitor_THT:C_Disc_D3.8mm_W2.6mm_P2.50mm
- C13: renamed from C7; footprint Capacitors_THT:C_Axial_L3.8mm_D2.6mm_P7.50mm_Horizontal -> Capacitor_THT:C_Disc_D3.8mm_W2.6mm_P2.50mm
- C14: renamed from C8; footprint Capacitors_THT:C_Axial_L3.8mm_D2.6mm_P7.50mm_Horizontal -> Capacitor_THT:C_Disc_D3.8mm_W2.6mm_P2.50mm
- C15: renamed from C9; footprint Capacitors_THT:C_Axial_L3.8mm_D2.6mm_P7.50mm_Horizontal -> Capacitor_THT:C_Disc_D3.8mm_W2.6mm_P2.50mm
- C16: renamed from C10; footprint Capacitors_THT:C_Axial_L3.8mm_D2.6mm_P7.50mm_Horizontal -> Capacitor_THT:C_Disc_D3.8mm_W2.6mm_P2.50mm
- C7: renamed from C1; value C -> 560pf; footprint Capacitors_THT:C_Axial_L3.8mm_D2.6mm_P7.50mm_Horizontal -> Capacitor_THT:C_Disc_D3.8mm_W2.6mm_P2.50mm
- C8: renamed from C2; footprint Capacitors_THT:C_Axial_L3.8mm_D2.6mm_P7.50mm_Horizontal -> Capacitor_THT:C_Disc_D3.8mm_W2.6mm_P2.50mm
- C9: renamed from C3; footprint Capacitors_THT:C_Axial_L3.8mm_D2.6mm_P7.50mm_Horizontal -> Capacitor_THT:C_Disc_D3.8mm_W2.6mm_P2.50mm
- D3: renamed from D1; footprint Diodes_THT:D_T-1_P5.08mm_Horizontal -> Diode_THT:D_DO-35_SOD27_P7.62mm_Horizontal
- D4: renamed from D2; footprint Diodes_THT:D_T-1_P5.08mm_Horizontal -> Diode_THT:D_DO-35_SOD27_P7.62mm_Horizontal
- H1: renamed from H2; footprint Mounting_Holes:MountingHole_2.2mm_M2 -> MountingHole:MountingHole_2.2mm_M2_DIN965_Pad
- H2: renamed from H1; footprint Mounting_Holes:MountingHole_2.2mm_M2 -> MountingHole:MountingHole_2.2mm_M2_DIN965_Pad
- J1: footprint Pin_Headers:Pin_Header_Straight_1x03_Pitch2.00mm -> Connector_PinHeader_2.00mm:PinHeader_1x03_P2.00mm_Vertical
- J2: renamed from J5; footprint Pin_Headers:Pin_Header_Straight_1x03_Pitch2.00mm -> Connector_PinHeader_2.00mm:PinHeader_1x03_P2.00mm_Vertical
- J3: renamed from J2; footprint Pin_Headers:Pin_Header_Straight_1x03_Pitch2.00mm -> Connector_PinHeader_2.00mm:PinHeader_1x03_P2.00mm_Vertical
- J4: renamed from J3; footprint Pin_Headers:Pin_Header_Straight_1x03_Pitch2.00mm -> Connector_PinHeader_2.00mm:PinHeader_1x03_P2.00mm_Vertical
- J5: renamed from J4; footprint Pin_Headers:Pin_Header_Straight_1x03_Pitch2.00mm -> Connector_PinHeader_2.00mm:PinHeader_1x03_P2.00mm_Vertical
- R15: renamed from R1; footprint Resistors_THT:R_Axial_DIN0204_L3.6mm_D1.6mm_P5.08mm_Horizontal -> Resistor_THT:R_Axial_DIN0207_L6.3mm_D2.5mm_P7.62mm_Horizontal
- R16: renamed from R2; footprint Resistors_THT:R_Axial_DIN0204_L3.6mm_D1.6mm_P5.08mm_Horizontal -> Resistor_THT:R_Axial_DIN0207_L6.3mm_D2.5mm_P7.62mm_Horizontal
- R17: renamed from R3; footprint Resistors_THT:R_Axial_DIN0204_L3.6mm_D1.6mm_P5.08mm_Horizontal -> Resistor_THT:R_Axial_DIN0207_L6.3mm_D2.5mm_P7.62mm_Horizontal
- R18: renamed from R4; footprint Resistors_THT:R_Axial_DIN0204_L3.6mm_D1.6mm_P5.08mm_Horizontal -> Resistor_THT:R_Axial_DIN0207_L6.3mm_D2.5mm_P7.62mm_Horizontal
- R19: renamed from R5; footprint Resistors_THT:R_Axial_DIN0204_L3.6mm_D1.6mm_P5.08mm_Horizontal -> Resistor_THT:R_Axial_DIN0207_L6.3mm_D2.5mm_P7.62mm_Horizontal
- R20: renamed from R6; footprint Resistors_THT:R_Axial_DIN0204_L3.6mm_D1.6mm_P5.08mm_Horizontal -> Resistor_THT:R_Axial_DIN0207_L6.3mm_D2.5mm_P7.62mm_Horizontal
- R21: renamed from R7; footprint Resistors_THT:R_Axial_DIN0204_L3.6mm_D1.6mm_P5.08mm_Horizontal -> Resistor_THT:R_Axial_DIN0207_L6.3mm_D2.5mm_P7.62mm_Horizontal
- R22: renamed from R8; footprint Resistors_THT:R_Axial_DIN0204_L3.6mm_D1.6mm_P5.08mm_Horizontal -> Resistor_THT:R_Axial_DIN0207_L6.3mm_D2.5mm_P7.62mm_Horizontal
- R23: renamed from R9; footprint Resistors_THT:R_Axial_DIN0204_L3.6mm_D1.6mm_P5.08mm_Horizontal -> Resistor_THT:R_Axial_DIN0207_L6.3mm_D2.5mm_P7.62mm_Horizontal
- R24: renamed from R10; footprint Resistors_THT:R_Axial_DIN0204_L3.6mm_D1.6mm_P5.08mm_Horizontal -> Resistor_THT:R_Axial_DIN0207_L6.3mm_D2.5mm_P7.62mm_Horizontal
- R25: renamed from R11; footprint Resistors_THT:R_Axial_DIN0204_L3.6mm_D1.6mm_P5.08mm_Horizontal -> Resistor_THT:R_Axial_DIN0207_L6.3mm_D2.5mm_P7.62mm_Horizontal
- R26: renamed from R12; footprint Resistors_THT:R_Axial_DIN0204_L3.6mm_D1.6mm_P5.08mm_Horizontal -> Resistor_THT:R_Axial_DIN0207_L6.3mm_D2.5mm_P7.62mm_Horizontal
- R27: renamed from R13; footprint Resistors_THT:R_Axial_DIN0204_L3.6mm_D1.6mm_P5.08mm_Horizontal -> Resistor_THT:R_Axial_DIN0207_L6.3mm_D2.5mm_P7.62mm_Horizontal
- R28: renamed from R14; footprint Resistors_THT:R_Axial_DIN0204_L3.6mm_D1.6mm_P5.08mm_Horizontal -> Resistor_THT:R_Axial_DIN0207_L6.3mm_D2.5mm_P7.62mm_Horizontal
- R29: renamed from R15; footprint Resistors_THT:R_Axial_DIN0204_L3.6mm_D1.6mm_P5.08mm_Horizontal -> Resistor_THT:R_Axial_DIN0207_L6.3mm_D2.5mm_P7.62mm_Horizontal
- R30: renamed from R22; footprint Resistors_THT:R_Axial_DIN0204_L3.6mm_D1.6mm_P5.08mm_Horizontal -> Resistor_THT:R_Axial_DIN0207_L6.3mm_D2.5mm_P7.62mm_Horizontal
- R31: renamed from R16; footprint Resistors_THT:R_Axial_DIN0204_L3.6mm_D1.6mm_P5.08mm_Horizontal -> Resistor_THT:R_Axial_DIN0207_L6.3mm_D2.5mm_P7.62mm_Horizontal
- R32: renamed from R23; footprint Resistors_THT:R_Axial_DIN0204_L3.6mm_D1.6mm_P5.08mm_Horizontal -> Resistor_THT:R_Axial_DIN0207_L6.3mm_D2.5mm_P7.62mm_Horizontal
- R33: renamed from R17; footprint Resistors_THT:R_Axial_DIN0204_L3.6mm_D1.6mm_P5.08mm_Horizontal -> Resistor_THT:R_Axial_DIN0207_L6.3mm_D2.5mm_P7.62mm_Horizontal
- R34: renamed from R24; footprint Resistors_THT:R_Axial_DIN0204_L3.6mm_D1.6mm_P5.08mm_Horizontal -> Resistor_THT:R_Axial_DIN0207_L6.3mm_D2.5mm_P7.62mm_Horizontal
- R35: renamed from R18; footprint Resistors_THT:R_Axial_DIN0204_L3.6mm_D1.6mm_P5.08mm_Horizontal -> Resistor_THT:R_Axial_DIN0207_L6.3mm_D2.5mm_P7.62mm_Horizontal
- R36: renamed from R19; footprint Resistors_THT:R_Axial_DIN0204_L3.6mm_D1.6mm_P5.08mm_Horizontal -> Resistor_THT:R_Axial_DIN0207_L6.3mm_D2.5mm_P7.62mm_Horizontal
- R37: renamed from R25; footprint Resistors_THT:R_Axial_DIN0204_L3.6mm_D1.6mm_P5.08mm_Horizontal -> Resistor_THT:R_Axial_DIN0207_L6.3mm_D2.5mm_P7.62mm_Horizontal
- R38: renamed from R26; footprint Resistors_THT:R_Axial_DIN0204_L3.6mm_D1.6mm_P5.08mm_Horizontal -> Resistor_THT:R_Axial_DIN0207_L6.3mm_D2.5mm_P7.62mm_Horizontal
- R39: renamed from R20; footprint Resistors_THT:R_Axial_DIN0204_L3.6mm_D1.6mm_P5.08mm_Horizontal -> Resistor_THT:R_Axial_DIN0207_L6.3mm_D2.5mm_P7.62mm_Horizontal
- R40: renamed from R21; footprint Resistors_THT:R_Axial_DIN0204_L3.6mm_D1.6mm_P5.08mm_Horizontal -> Resistor_THT:R_Axial_DIN0207_L6.3mm_D2.5mm_P7.62mm_Horizontal
- RV2: renamed from RV1; footprint Potentiometers:Potentiometer_WirePads_Small -> Potentiometer_THT:Potentiometer_ACP_CA9-H2,5_Horizontal
- RV3: renamed from RV2; footprint Potentiometers:Potentiometer_WirePads_Small -> Potentiometer_THT:Potentiometer_ACP_CA9-H2,5_Horizontal
- RV4: renamed from RV3; footprint Potentiometers:Potentiometer_WirePads_Small -> Potentiometer_THT:Potentiometer_ACP_CA9-H2,5_Horizontal
- RV5: renamed from RV4; footprint Potentiometers:Potentiometer_WirePads_Small -> Potentiometer_THT:Potentiometer_ACP_CA9-H2,5_Horizontal
- U2: renamed from U1; footprint LF351N:DIP254P762X533-8 -> Package_DIP:DIP-8_W7.62mm_LongPads; symbol 2019-03-05_16-55-55:LF353N -> Pre-amp-rescue:LF353N-2019-03-05_16-55-55
- U3: renamed from U2; footprint LF351N:DIP254P762X533-8 -> Package_DIP:DIP-8_W7.62mm_LongPads; symbol 2019-03-05_16-55-55:LF353N -> Pre-amp-rescue:LF353N-2019-03-05_16-55-55
- U4: renamed from U3; footprint LF351N:DIP254P762X533-8 -> Package_DIP:DIP-8_W7.62mm_LongPads; symbol 2019-03-05_16-55-55:LF353N -> Pre-amp-rescue:LF353N-2019-03-05_16-55-55
Connections:
- wire segments 169 -> 236
Other:
- moved on the sheet: C10, C11, C12, C13, C14, C15, C16, C7, C8, C9, D3, D4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

Commit message: update version
Other:
- moved on the sheet: H2
Changed lines of the file:
@@
 EESchema Schematic File Version 4
 LIBS:Pre-amp-cache
-EELAYER 26 0
+EELAYER 29 0
 EELAYER END
 $Descr B 17000 11000
@@
 Sheet 1 1
 Title "preamp"
-Date "2019-03-12"
-Rev "1.0"
+Date "2019-04-01"
+Rev "1.1.1"
 Comp "MXM Designs"
 Comment1 ""
@@
 L Mechanical:MountingHole H2
 U 1 1 5C81F472
-P 16350 600
-F 0 "H2" H 16450 646 50  0000 L CNN
-F 1 "MountingHole" H 16450 555 50  0000 L CNN
-F 2 "MountingHole:MountingHole_2.2mm_M2_DIN965_Pad" H 16350 600 50  0001 C CNN
-F 3 "~" H 16350 600 50  0001 C CNN
-	1    16350 600
-	1    0    0    -1
-$EndComp
+P 650 1600
+F 0 "H2" H 750 1646 50  0000 L CNN
+F 1 "MountingHole" H 750 1555 50  0000 L CNN
+F 2 "MountingHole:MountingHole_2.2mm_M2_DIN965_Pad" H 650 1600 50  0001 C CNN
+F 3 "~" H 650 1600 50  0001 C CNN
+	1    650  1600
+	1    0    0    -1
+$EndComp

Commit message: update to pc mount pots
Parts:
- RV1, RV2, RV3, RV4, RV5: footprint Potentiometer_THT:Potentiometer_ACP_CA9-H2,5_Horizontal -> Potentiometers:Potentiometer_Alps_RK163_Single_Vertical
Changed lines of the file:
@@
 F 0 "RV2" V 7795 4600 50  0000 C CNN
 F 1 "25k-L" V 7886 4600 50  0000 C CNN
-F 2 "Potentiometer_THT:Potentiometer_ACP_CA9-H2,5_Horizontal" H 8000 4600 50  0001 C CNN
+F 2 "Potentiometers:Potentiometer_Alps_RK163_Single_Vertical" H 8000 4600 50  0001 C CNN
 F 3 "~" H 8000 4600 50  0001 C CNN
 	1    8000 4600
@@
 F 0 "RV3" V 9545 3650 50  0000 C CNN
 F 1 "25k-A" V 9636 3650 50  0000 C CNN
-F 2 "Potentiometer_THT:Potentiometer_ACP_CA9-H2,5_Horizontal" H 9750 3650 50  0001 C CNN
+F 2 "Potentiometers:Potentiometer_Alps_RK163_Single_Vertical" H 9750 3650 50  0001 C CNN
 F 3 "~" H 9750 3650 50  0001 C CNN
 	1    9750 3650
@@
 F 0 "RV4" V 11145 4650 50  0000 C CNN
 F 1 "25k-L" V 11236 4650 50  0000 C CNN
-F 2 "Potentiometer_THT:Potentiometer_ACP_CA9-H2,5_Horizontal" H 11350 4650 50  0001 C CNN
+F 2 "Potentiometers:Potentiometer_Alps_RK163_Single_Vertical" H 11350 4650 50  0001 C CNN
 F 3 "~" H 11350 4650 50  0001 C CNN
 	1    11350 4650
@@
 F 0 "RV5" V 12945 4650 50  0000 C CNN
 F 1 "25k-L" V 13036 4650 50  0000 C CNN
-F 2 "Potentiometer_THT:Potentiometer_ACP_CA9-H2,5_Horizontal" H 13150 4650 50  0001 C CNN
+F 2 "Potentiometers:Potentiometer_Alps_RK163_Single_Vertical" H 13150 4650 50  0001 C CNN
 F 3 "~" H 13150 4650 50  0001 C CNN
 	1    13150 4650
@@
 F 0 "RV1" V 6495 5400 50  0000 C CNN
 F 1 "25k-L" V 6586 5400 50  0000 C CNN
-F 2 "Potentiometer_THT:Potentiometer_ACP_CA9-H2,5_Horizontal" H 6700 5400 50  0001 C CNN
+F 2 "Potentiometers:Potentiometer_Alps_RK163_Single_Vertical" H 6700 5400 50  0001 C CNN
 F 3 "~" H 6700 5400 50  0001 C CNN
 	1    6700 5400

Commit message: create new branch  1.1.4
Parts:
- removed C6: 10, Capacitor_THT:C_Disc_D3.8mm_W2.6mm_P2.50mm, symbol Device:C
- added C6: 10uF, Capacitor_THT:CP_Radial_D4.0mm_P1.50mm, symbol Device:CP
- C14: value .47 -> .047
- R2: value 23k -> 22k
- R3: Manufacturer (none) -> Royal Ohm; tolerance (none) -> 1%; type (none) -> metal film
Connections:
- net GND: now also D2.2 (A), U4.5 (IN+); no longer D2.1 (K)
- net at D1.1 (K): now also D2.1 (K); no longer D2.2 (A)
- net at R37.1, U4.3 (IN+): now also D3.1 (K); no longer D3.2 (A)
- net at U4.6 (IN-): now also U4.7 (OUT)
- net at D4.2 (A): now also D3.2 (A); no longer D3.1 (K)
- net at R8.1, R9.2: now also R10.1, R11.2
- net at R12.1: now also C6.1
- net at RV1.3: now also C6.2
- no-connect marks 6 -> 3
Changed lines of the file:
@@
 Sheet 1 1
 Title "preamp"
-Date "2019-04-01"
-Rev "1.1.1"
+Date "2019-04-27"
+Rev "1.1.4"
 Comp "MXM Designs"
 Comment1 ""
@@
 F 1 "220K" V 9234 5400 50  0000 C CNN
 F 2 "Resistor_THT:R_Axial_DIN0207_L6.3mm_D2.5mm_P7.62mm_Horizontal" V 9280 5400 50  0001 C CNN
-F 3 "~" H 9350 5400 50  0001 C CNN
+F 3 "https://www.taydaelectronics.com/datasheets/files/royalohmprecisionmetalmf.pdf" H 9350 5400 50  0001 C CNN
 	1    9350 5400
 	0    1    1    0
@@
 F 1 "220K" V 10034 5400 50  0000 C CNN
 F 2 "Resistor_THT:R_Axial_DIN0207_L6.3mm_D2.5mm_P7.62mm_Horizontal" V 10080 5400 50  0001 C CNN
-F 3 "~" H 10150 5400 50  0001 C CNN
+F 3 "https://www.taydaelectronics.com/datasheets/files/royalohmprecisionmetalmf.pdf" H 10150 5400 50  0001 C CNN
 	1    10150 5400
 	0    1    1    0
@@
 F 1 "220K" V 10784 5400 50  0000 C CNN
 F 2 "Resistor_THT:R_Axial_DIN0207_L6.3mm_D2.5mm_P7.62mm_Horizontal" V 10830 5400 50  0001 C CNN
-F 3 "~" H 10900 5400 50  0001 C CNN
+F 3 "https://www.taydaelectronics.com/datasheets/files/royalohmprecisionmetalmf.pdf" H 10900 5400 50  0001 C CNN
 	1    10900 5400
 	0    1    1    0
@@
 F 1 "220K" V 11634 5400 50  0000 C CNN
 F 2 "Resistor_THT:R_Axial_DIN0207_L6.3mm_D2.5mm_P7.62mm_Horizontal" V 11680 5400 50  0001 C CNN
-F 3 "~" H 11750 5400 50  0001 C CNN
+F 3 "https://www.taydaelectronics.com/datasheets/files/royalohmprecisionmetalmf.pdf" H 11750 5400 50  0001 C CNN
 	1    11750 5400
 	0    1    1    0
@@
 F 1 "220K" V 12634 5400 50  0000 C CNN
 F 2 "Resistor_THT:R_Axial_DIN0207_L6.3mm_D2.5mm_P7.62mm_Horizontal" V 12680 5400 50  0001 C CNN
-F 3 "~" H 12750 5400 50  0001 C CNN
+F 3 "https://www.taydaelectronics.com/datasheets/files/royalohmprecisionmetalmf.pdf" H 12750 5400 50  0001 C CNN
 	1    12750 5400
 	0    1    1    0
@@
 F 1 "220K" V 13534 5400 50  0000 C CNN
 F 2 "Resistor_THT:R_Axial_DIN0207_L6.3mm_D2.5mm_P7.62mm_Horizontal" V 13580 5400 50  0001 C CNN
-F 3 "~" H 13650 5400 50  0001 C CNN
+F 3 "https://www.taydaelectronics.com/datasheets/files/royalohmprecisionmetalmf.pdf" H 13650 5400 50  0001 C CNN
 	1    13650 5400
 	0    1    1    0
@@
 P 13150 5150
 F 0 "C14" H 13265 5196 50  0000 L CNN
-F 1 ".47" H 13265 5105 50  0000 L CNN
+F 1 ".047" H 13265 5105 50  0000 L CNN
 F 2 "Capacitor_THT:C_Disc_D3.8mm_W2.6mm_P2.50mm" H 13188 5000 50  0001 C CNN
 F 3 "~" H 13150 5150 50  0001 C CNN
@@
 F 3 "~" H 13800 7350 50  0001 C CNN
 	1    13800 7350
-	0    -1   -1   0
+	0    1    1    0
 $EndComp
 $Comp
@@
 	13000 7450 13000 7300
 Connection ~ 12350 7850
-NoConn ~ 11400 7000
-NoConn ~ 11400 7100
-NoConn ~ 11400 7200
 $Comp
 L Connector:Barrel_Jack_Switch J1
@@
 P 2050 5000
 F 0 "R2" V 1843 5000 50  0000 C CNN
-F 1 "23k" V 1934 5000 50  0000 C CNN
+F 1 "22k" V 1934 5000 50  0000 C CNN
 F 2 "Resistor_THT:R_Axial_DIN0207_L6.3mm_D2.5mm_P7.62mm_Horizontal" V 1980 5000 50  0001 C CNN
 F 3 "~" H 2050 5000 50  0001 C CNN
@@
 F 1 "3.3k" H 4380 7095 50  0000 R CNN
 F 2 "Resistor_THT:R_Axial_DIN0207_L6.3mm_D2.5mm_P7.62mm_Horizontal" V 4380 7050 50  0001 C CNN
-F 3 "~" H 4450 7050 50  0001 C CNN
+F 3 "https://www.taydaelectronics.com/datasheets/files/royalohmprecisionmetalmf.pdf" H 4450 7050 50  0001 C CNN
 	1    4450 7050
 	-1   0    0    1
@@
 F 1 "220k" H 3030 6245 50  0000 R CNN
 F 2 "Resistor_THT:R_Axial_DIN0207_L6.3mm_D2.5mm_P7.62mm_Horizontal" V 3030 6200 50  0001 C CNN
-F 3 "~" H 3100 6200 50  0001 C CNN
+F 3 "https://www.taydaelectronics.com/datasheets/files/royalohmprecisionmetalmf.pdf" H 3100 6200 50  0001 C CNN
+F 4 "metal film" H 3100 6200 50  0001 C CNN "type"
+F 5 "1%" H 3100 6200 50  0001 C CNN "tolerance"
+F 6 "Royal Ohm" H 3100 6200 50  0001 C CNN "Manufacturer"
 	1    3100 6200
 	-1   0    0    1
@@
 F 3 "~" H 2300 6550 50  0001 C CNN
 	1    2300 6550
-	0    -1   -1   0
+	0    1    1    0
 $EndComp
 $Comp
@@
 F 1 "33k" V 3800 6450 50  0000 C CNN
 F 2 "Resistor_THT:R_Axial_DIN0207_L6.3mm_D2.5mm_P7.62mm_Horizontal" V 3830 6450 50  0001 C CNN
-F 3 "~" H 3900 6450 50  0001 C CNN
+F 3 "https://www.taydaelectronics.com/datasheets/files/royalohmprecisionmetalmf.pdf" H 3900 6450 50  0001 C CNN
 	1    3900 6450
 	0    -1   -1   0
@@
 F 1 "3.3k" H 3330 6845 50  0000 R CNN
 F 2 "Resistor_THT:R_Axial_DIN0207_L6.3mm_D2.5mm_P7.62mm_Horizontal" V 3330 6800 50  0001 C CNN
-F 3 "~" H 3400 6800 50  0001 C CNN
+F 3 "https://www.taydaelectronics.com/datasheets/files/royalohmprecisionmetalmf.pdf" H 3400 6800 50  0001 C CNN
 	1    3400 6800
 	-1   0    0    1
@@
 F 1 "22k" H 4380 7495 50  0000 R CNN
 F 2 "Resistor_THT:R_Axial_DIN0207_L6.3mm_D2.5mm_P7.62mm_Horizontal" V 4380 7450 50  0001 C CNN
-F 3 "~" H 4450 7450 50  0001 C CNN
+F 3 "https://www.taydaelectronics.com/datasheets/files/royalohmprecisionmetalmf.pdf" H 4450 7450 50  0001 C CNN
 	1    4450 7450
 	-1   0    0    1
@@
 F 1 "12k" H 4880 7595 50  0000 R CNN
 F 2 "Resistor_THT:R_Axial_DIN0207_L6.3mm_D2.5mm_P7.62mm_Horizontal" V 4880 7550 50  0001 C CNN
-F 3 "~" H 4950 7550 50  0001 C CNN
+F 3 "https://www.taydaelectronics.com/datasheets/files/royalohmprecisionmetalmf.pdf" H 4950 7550 50  0001 C CNN
 	1    4950 7550
 	-1   0    0    1
@@
 F 1 "1k" H 4880 7995 50  0000 R CNN
 F 2 "Resistor_THT:R_Axial_DIN0207_L6.3mm_D2.5mm_P7.62mm_Horizontal" V 4880 7950 50  0001 C CNN
-F 3 "~" H 4950 7950 50  0001 C CNN
+F 3 "https://www.taydaelectronics.com/datasheets/files/royalohmprecisionmetalmf.pdf" H 4950 7950 50  0001 C CNN
 	1    4950 7950
 	-1   0    0    1
@@
 	4950 8650 4950 8500
 Wire Wire Line
-	4950 7700 4950 7800
+	4950 7700 4950 7750
 $Comp
 L Device:R R10
@@
 F 1 "22k" H 5480 7595 50  0000 R CNN
 F 2 "Resistor_THT:R_Axial_DIN0207_L6.3mm_D2.5mm_P7.62mm_Horizontal" V 5480 7550 50  0001 C CNN
-F 3 "~" H 5550 7550 50  0001 C CNN
+F 3 "https://www.taydaelectronics.com/datasheets/files/royalohmprecisionmetalmf.pdf" H 5550 7550 50  0001 C CNN
 	1    5550 7550
 	-1   0    0    1
@@
 F 1 "22k" H 5480 7995 50  0000 R CNN
 F 2 "Resistor_THT:R_Axial_DIN0207_L6.3mm_D2.5mm_P7.62mm_Horizontal" V 5480 7950 50  0001 C CNN
-F 3 "~" H 5550 7950 50  0001 C CNN
+F 3 "https://www.taydaelectronics.com/datasheets/files/royalohmprecisionmetalmf.pdf" H 5550 7950 50  0001 C CNN
 	1    5550 7950
 	-1   0    0    1
@@
 $EndComp
 Wire Wire Line
-	5550 7700 5550 7800
+	5550 7700 5550 7750
 Wire Wire Line
 	5550 8100 5550 8650
@@
 F 1 "82k" V 5734 5750 50  0000 C CNN
 F 2 "Resistor_THT:R_Axial_DIN0207_L6.3mm_D2.5mm_P7.62mm_Horizontal" V 5780 5750 50  0001 C CNN
-F 3 "~" H 5850 5750 50  0001 C CNN
+F 3 "https://www.taydaelectronics.com/datasheets/files/royalohmprecisionmetalmf.pdf" H 5850 5750 50  0001 C CNN
 	1    5850 5750
 	0    1    1    0
@@
 F 1 "1k" V 5734 5400 50  0000 C CNN
 F 2 "Resistor_THT:R_Axial_DIN0207_L6.3mm_D2.5mm_P7.62mm_Horizontal" V 5780 5400 50  0001 C CNN
-F 3 "~" H 5850 5400 50  0001 C CNN
+F 3 "https://www.taydaelectronics.com/datasheets/files/royalohmprecisionmetalmf.pdf" H 5850 5400 50  0001 C CNN
 	1    5850 5400
 	0    1    1    0
@@
 Wire Wire Line
 	5650 5750 5100 5750
-$Comp
-L Device:C C6
-U 1 1 5CAA9690
-P 6250 5400
-F 0 "C6" V 6100 5400 50  0000 C CNN
-F 1 "10" V 6400 5400 50  0000 C CNN
-F 2 "Capacitor_THT:C_Disc_D3.8mm_W2.6mm_P2.50mm" H 6288 5250 50  0001 C CNN
-F 3 "~" H 6250 5400 50  0001 C CNN
-	1    6250 5400
-	0    -1   -1   0
-$EndComp
 Wire Wire Line
 	6000 5400 6100 5400
@@
 F 1 "3.3k" V 6234 5850 50  0000 C CNN
 F 2 "Resistor_THT:R_Axial_DIN0207_L6.3mm_D2.5mm_P7.62mm_Horizontal" V 6280 5850 50  0001 C CNN
-F 3 "~" H 6350 5850 50  0001 C CNN
+F 3 "https://www.taydaelectronics.com/datasheets/files/royalohmprecisionmetalmf.pdf" H 6350 5850 50  0001 C CNN
 	1    6350 5850
 	0    1    1    0
@@
 	1    0    0    -1
 $EndComp
+$Comp
+L power:GND #PWR0101
+U 1 1 5CDA41BF
+P 10500 7100
+F 0 "#PWR0101" H 10500 6850 50  0001 C CNN
+F 1 "GND" H 10505 6927 50  0000 C CNN
+F 2 "" H 10500 7100 50  0001 C CNN
+F 3 "" H 10500 7100 50  0001 C CNN
+	1    10500 7100
+	1    0    0    -1
+$EndComp
+Wire Wire Line
+	11400 7000 10500 7000
+Wire Wire Line
+	10500 7000 10500 7100
+Wire Wire Line
+	11250 7200 11250 7100
+Wire Wire Line
+	11250 7100 11400 7100
+Wire Wire Line
+	11400 7200 11250 7200
+$Comp
+L Device:CP C6
+U 1 1 5CE51529
+P 6250 5400
+F 0 "C6" V 6505 5400 50  0000 C CNN
+F 1 "10uF" V 6414 5400 50  0000 C CNN
+F 2 "Capacitor_THT:CP_Radial_D4.0mm_P1.50mm" H 6288 5250 50  0001 C CNN
+F 3 "~" H 6250 5400 50  0001 C CNN
+	1    6250 5400
+	0    -1   -1   0
+$EndComp
+Wire Wire Line
+	5550 7750 4950 7750
+Connection ~ 5550 7750
+Wire Wire Line
+	5550 7750 5550 7800
+Connection ~ 4950 7750
+Wire Wire Line
+	4950 7750 4950 7800
 $EndSCHEMATC
