File: IOBoard/IOBoard.kicad_pcb (KiCad board)
At the start: 2 copper layers, 281.9 x 22.9 mm, 24 parts, among them J1 IN, J10 Conn_01x06_Male, J2 In2, J3 Send, J4 Conn_01x24_Male, J5 Return, J6 Out, J7 A/B, J8 Conn_01x10_Male, J9 Conn_01x05_Male

Commit message: add jacks
Parts:
- removed the J7 at (285.8, 52.1)
- added J4: RA49C12A, RA49C12A:RA49C14B, F.Cu at (268.0, 57.1)
- J1: value IN -> RA49C12A; footprint Connector_Audio:Jack_3.5mm_QingPu_WQP-PJ398SM_Vertical_CircularHoles -> RA49C12A:RA49C14B
- J2: value In2 -> RA49C12A; footprint Connector_Audio:Jack_3.5mm_QingPu_WQP-PJ398SM_Vertical_CircularHoles -> RA49C12A:RA49C14B
- J3: value Send -> RA49C12A; footprint Connector_Audio:Jack_3.5mm_QingPu_WQP-PJ398SM_Vertical_CircularHoles -> RA49C12A:RA49C14B
- J5: value Return -> RA49C12A; footprint Connector_Audio:Jack_3.5mm_QingPu_WQP-PJ398SM_Vertical_CircularHoles -> RA49C12A:RA49C14B
- J6: value Out -> RA49C12A; footprint Connector_Audio:Jack_3.5mm_QingPu_WQP-PJ398SM_Vertical_CircularHoles -> RA49C12A:RA49C14B
- moved H1 44.0 mm to (55.9, 78.1)
- moved J7 35.0 mm to (226.2, 76.2)
- moved J6 30.9 mm to (304.8, 57.1), turned to 90 degrees
- moved J5 24.0 mm to (286.4, 57.1), turned to 90 degrees
- moved J1 16.5 mm to (0.64, 56.5), turned to 90 degrees
- moved J2 9.93 mm to (19.1, 56.5), turned to 90 degrees
- moved J8 6.38 mm to (36.2, 77.5)
- moved J3 5.43 mm to (249.6, 57.1), turned to 90 degrees
- renumbered J9 to J10, J8 to J7, J10 to J8, J4 to J9
Connections:
- J7 pad 1: Net-(J3-PadT) -> Net-(J3-Pad1)
- J7 pad 10: Net-(J7-PadS) -> Net-(J6-Pad2)
- J7 pad 2: Net-(J3-PadS) -> Net-(J3-Pad5)
- J7 pad 3: Net-(J5-PadTN) -> Net-(J4-Pad1)
- J7 pad 4: Net-(J5-PadT) -> Net-(J4-Pad5)
- J7 pad 5: Net-(J5-PadS) -> Net-(J4-Pad2)
- J7 pad 6: Net-(J6-PadT) -> Net-(J5-Pad1)
- J7 pad 7: Net-(J6-PadS) -> Net-(J5-Pad5)
- J7 pad 8: Net-(J7-PadTN) -> Net-(J6-Pad1)
- J7 pad 9: Net-(J7-PadT) -> Net-(J6-Pad5)
- J8 pad 1: Net-(J1-PadTN) -> Net-(J1-Pad1)
- J8 pad 2: Net-(J1-PadT) -> GND
- J8 pad 3: Net-(J1-PadS) -> Net-(J1-Pad2)
- J8 pad 4: Net-(J10-Pad4) -> Net-(J2-Pad1)
- J8 pad 5: Net-(J10-Pad5) -> Net-(J2-Pad5)
- J8 pad 6: Net-(J10-Pad6) -> Net-(J2-Pad2)
Routing:
- net Net-(J1-PadS): track 37.6 -> 0.00 mm
- net Net-(J10-Pad4): track 32.4 -> 0.00 mm
- net Net-(J1-PadTN): track 32.0 -> 0.00 mm
- net Net-(J10-Pad6): track 30.0 -> 0.00 mm
- net Net-(J7-PadS): track 28.7 -> 0.00 mm
- net Net-(J3-PadS): track 27.9 -> 0.00 mm
- net Net-(J1-PadT): track 27.9 -> 0.00 mm
- net (no net): track 0.00 -> 25.0 mm
- net Net-(J10-Pad5): track 23.9 -> 0.00 mm
- net Net-(J5-PadS): track 23.0 -> 0.00 mm
- net Net-(J6-PadS): track 21.8 -> 0.00 mm
- net Net-(J7-PadTN): track 21.0 -> 0.00 mm
- net Net-(J5-PadTN): track 18.9 -> 0.00 mm
- net Net-(J3-PadT): track 16.0 -> 0.00 mm
- net Net-(J7-PadT): track 14.0 -> 0.00 mm
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Other:
- board size 281.9 x 22.9 mm -> 327 x 29.8 mm

Commit message: split connectors and reflow
Parts:
- added J11: Conn_01x12_Male, Connector_PinHeader_2.00mm:PinHeader_1x12_P2.00mm_Vertical, F.Cu at (238.8, 229.9)
- J9: value Conn_01x24_Male -> Conn_01x12_Male; footprint Connector_PinHeader_2.00mm:PinHeader_1x24_P2.00mm_Vertical -> Connector_PinHeader_2.00mm:PinHeader_1x12_P2.00mm_Vertical
- moved R1 167.1 mm to (116.8, 212.7)
- moved J8 166.1 mm to (102.2, 229.9)
- moved J10 166.0 mm to (131.4, 229.9)
- moved RV8 165.3 mm to (299.7, 209.6)
- moved J1 165.3 mm to (61.6, 210.2)
- moved J2 165.3 mm to (80.0, 210.2)
- moved J7 165.3 mm to (287.2, 229.9)
- moved RV6 165.3 mm to (248.9, 209.6)
- moved RV7 165.3 mm to (274.3, 209.6)
- moved D1 165.3 mm to (116.8, 207.0)
- moved D2 165.3 mm to (144.8, 207.0)
- moved R2 165.3 mm to (144.8, 210.8)
- moved J5 164.7 mm to (347.3, 210.2)
- moved J3 164.7 mm to (310.5, 210.2)
- moved J4 164.7 mm to (328.9, 210.2)
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Connections:
- J7 pad 1: Net-(J3-Pad1) -> Net-(J4-Pad5)
- J7 pad 4: Net-(J4-Pad5) -> Net-(J3-Pad1)
- J7 pad 8: Net-(J6-Pad1) -> Net-(J6-Pad5)
- J7 pad 9: Net-(J6-Pad5) -> Net-(J6-Pad1)
- J8 pad 5: Net-(J2-Pad5) -> Net-(J2-Pad2)
- J8 pad 6: Net-(J2-Pad2) -> Net-(J2-Pad5)
- RV5 pad 1: Net-(J9-Pad15) -> Net-(J11-Pad3)
- RV5 pad 2: Net-(J9-Pad14) -> Net-(J11-Pad2)
- RV5 pad 3: Net-(J9-Pad13) -> Net-(J11-Pad1)
- RV6 pad 1: Net-(J9-Pad18) -> Net-(J11-Pad6)
- RV6 pad 2: Net-(J9-Pad17) -> Net-(J11-Pad5)
- RV6 pad 3: Net-(J9-Pad16) -> Net-(J11-Pad4)
- RV7 pad 1: Net-(J9-Pad21) -> Net-(J11-Pad9)
- RV7 pad 2: Net-(J9-Pad20) -> Net-(J11-Pad8)
- RV7 pad 3: Net-(J9-Pad19) -> Net-(J11-Pad7)
- RV8 pad 1: Net-(J9-Pad24) -> Net-(J11-Pad12)
- RV8 pad 2: Net-(J9-Pad23) -> Net-(J11-Pad11)
- RV8 pad 3: Net-(J9-Pad22) -> Net-(J11-Pad10)
Routing:
- net Net-(J6-Pad2): track 6.13 -> 84.5 mm
- net Net-(J9-Pad24): track 77.2 -> 0.00 mm
- net Net-(J9-Pad23): track 74.2 -> 0.00 mm
- net Net-(J9-Pad22): track 70.6 -> 0.00 mm
- net Net-(J6-Pad5): track 3.69 -> 73.3 mm
- net Net-(J6-Pad1): track 0.00 -> 68.1 mm
- net Net-(J5-Pad5): track 0.00 -> 67.7 mm
- net Net-(J9-Pad21): track 57.8 -> 0.00 mm
- net Net-(J5-Pad1): track 0.00 -> 55.2 mm
- net Net-(J9-Pad20): track 54.8 -> 0.00 mm
- net Net-(J11-Pad8): track 0.00 -> 53.2 mm
- net Net-(J4-Pad5): track 0.00 -> 52.8 mm
- net Net-(J9-Pad19): track 51.8 -> 0.00 mm
- net Net-(J11-Pad12): track 0.00 -> 47.4 mm
- net Net-(J4-Pad2): track 0.95 -> 46.3 mm
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Other:
- board size 327 x 29.8 mm -> 323.2 x 29.8 mm

Commit message: move to the same size connectors
Parts:
- J10: value Conn_01x05_Male -> Conn_01x08_Male; footprint Connector_PinHeader_2.00mm:PinHeader_1x05_P2.00mm_Vertical -> Connector_JST:JST_PH_B8B-PH-K_1x08_P2.00mm_Vertical
- J11, J9: value Conn_01x12_Male -> Conn_01x08_Male; footprint Connector_PinHeader_2.00mm:PinHeader_1x12_P2.00mm_Vertical -> Connector_JST:JST_PH_B8B-PH-K_1x08_P2.00mm_Vertical
- J7: value Conn_01x10_Male -> Conn_01x08_Male; footprint Connector_PinHeader_2.00mm:PinHeader_1x10_P2.00mm_Vertical -> Connector_JST:JST_PH_B8B-PH-K_1x08_P2.00mm_Vertical
- J8: value Conn_01x06_Male -> Conn_01x08_Male; footprint Connector_PinHeader_2.00mm:PinHeader_1x06_P2.00mm_Vertical -> Connector_JST:JST_PH_B8B-PH-K_1x08_P2.00mm_Vertical
- moved J10 61.6 mm to (193.0, 228.6), turned to 0 degrees
- moved J8 5.85 mm to (96.5, 228.6), turned to 0 degrees
- moved J11 2.84 mm to (241.3, 228.6), turned to 0 degrees
- moved J7 2.70 mm to (289.6, 228.6), turned to 0 degrees
- moved J9 1.64 mm to (144.8, 228.6), turned to 0 degrees
Connections:
- J1 pad 3: (no net) -> Net-(J1-Pad3)
- J1 pad 4: (no net) -> Net-(J1-Pad4)
- J1 pad 6: (no net) -> Net-(J1-Pad6)
- J10 pad 1: GND -> Net-(J10-Pad1)
- J10 pad 2: Net-(D2-Pad2) -> Net-(J10-Pad2)
- J10 pad 3: Net-(D1-Pad2) -> Net-(J10-Pad3)
- J10 pad 4: (no net) -> Net-(J10-Pad4)
- J10 pad 5: (no net) -> Net-(J10-Pad5)
- J2 pad 3: (no net) -> Net-(J2-Pad3)
- J2 pad 4: (no net) -> Net-(J2-Pad4)
- J2 pad 6: (no net) -> Net-(J2-Pad6)
- J3 pad 2: (no net) -> Net-(J3-Pad2)
- J3 pad 3: (no net) -> Net-(J3-Pad3)
- J3 pad 4: (no net) -> Net-(J3-Pad4)
- J3 pad 5: Net-(J3-Pad5) -> Net-(J11-Pad8)
- J3 pad 6: (no net) -> Net-(J3-Pad6)
- J4 pad 3: (no net) -> Net-(J4-Pad3)
- J4 pad 4: (no net) -> Net-(J4-Pad4)
- J4 pad 5: Net-(J4-Pad5) -> Net-(J11-Pad7)
- J4 pad 6: (no net) -> Net-(J4-Pad6)
- J5 pad 2: (no net) -> Net-(J5-Pad2)
- J5 pad 3: (no net) -> Net-(J5-Pad3)
- J5 pad 4: (no net) -> Net-(J5-Pad4)
- J5 pad 6: (no net) -> Net-(J5-Pad6)
- J6 pad 3: (no net) -> Net-(J6-Pad3)
- J6 pad 4: (no net) -> Net-(J6-Pad4)
- J6 pad 6: (no net) -> Net-(J6-Pad6)
- J7 pad 1: Net-(J4-Pad5) -> Net-(J4-Pad1)
- J7 pad 2: Net-(J3-Pad5) -> Net-(J3-Pad1)
- J7 pad 3: Net-(J4-Pad1) -> Net-(J4-Pad2)
- J7 pad 4: Net-(J3-Pad1) -> Net-(J5-Pad1)
- J7 pad 5: Net-(J4-Pad2) -> Net-(J5-Pad5)
- J7 pad 6: Net-(J5-Pad1) -> Net-(J6-Pad5)
- J7 pad 7: Net-(J5-Pad5) -> Net-(J6-Pad1)
- J7 pad 8: Net-(J6-Pad5) -> Net-(J6-Pad2)
- J9 pad 1: Net-(J9-Pad1) -> +15V
- J9 pad 2: GND -> Net-(J9-Pad2)
- J9 pad 3: Net-(J9-Pad3) -> GND
- J9 pad 4: GND -> Net-(J9-Pad4)
- J9 pad 7: GND -> Net-(J9-Pad7)
- RV1 pad 1: Net-(J9-Pad3) -> Net-(J9-Pad4)
- RV1 pad 3: Net-(J9-Pad1) -> Net-(J9-Pad2)
- RV3 pad 1: Net-(J9-Pad9) -> Net-(J9-Pad8)
- RV3 pad 2: Net-(J9-Pad8) -> Net-(J9-Pad7)
- RV4 pad 1: Net-(J9-Pad12) -> Net-(J10-Pad2)
- RV4 pad 2: Net-(J9-Pad11) -> Net-(J10-Pad1)
- RV5 pad 1: Net-(J11-Pad3) -> Net-(J10-Pad5)
- RV5 pad 2: Net-(J11-Pad2) -> Net-(J10-Pad4)
- RV5 pad 3: Net-(J11-Pad1) -> Net-(J10-Pad3)
- RV6 pad 1: Net-(J11-Pad6) -> Net-(J10-Pad8)
- RV6 pad 2: Net-(J11-Pad5) -> Net-(J10-Pad7)
- RV6 pad 3: Net-(J11-Pad4) -> Net-(J10-Pad6)
- RV7 pad 1: Net-(J11-Pad9) -> Net-(J11-Pad3)
- RV7 pad 2: Net-(J11-Pad8) -> Net-(J11-Pad2)
- RV7 pad 3: Net-(J11-Pad7) -> Net-(J11-Pad1)
- RV8 pad 1: Net-(J11-Pad12) -> Net-(J11-Pad6)
- RV8 pad 2: Net-(J11-Pad11) -> Net-(J11-Pad5)
- RV8 pad 3: Net-(J11-Pad10) -> Net-(J11-Pad4)
Routing:
- net Net-(J9-Pad4): track 0.00 -> 88.6 mm
- net Net-(J11-Pad7): track 25.9 -> 86.9 mm
- net Net-(J9-Pad2): track 0.00 -> 56.2 mm
- net Net-(J9-Pad1): track 54.1 -> 0.00 mm
- net Net-(J4-Pad5): track 52.8 -> 0.00 mm
- net Net-(J10-Pad8): track 0.00 -> 52.2 mm
- net Net-(J9-Pad3): track 50.1 -> 0.00 mm
- net Net-(J10-Pad7): track 0.00 -> 49.2 mm
- net Net-(J11-Pad12): track 47.4 -> 0.00 mm
- net Net-(J10-Pad6): track 0.00 -> 45.2 mm
- net Net-(J11-Pad11): track 44.4 -> 0.00 mm
- net Net-(J11-Pad10): track 41.4 -> 0.00 mm
- net Net-(J9-Pad12): track 36.4 -> 0.00 mm
- net Net-(J11-Pad6): track 20.4 -> 56.5 mm
- net Net-(J9-Pad11): track 33.4 -> 0.00 mm
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